Commit message: rm token

File: rocap_ros/urdf/rocap/rocap.urdf (robot description, URDF)
Before this commit: robot rocap, 34 links, 33 joints
Links:
- added link rocap_body, mass 0.001; collision box size=0.4 0.4 0.45; visual mesh filename=file:///home/oli/ros2_ws/install/rocap_ros/share/rocap_ros/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 scale=0.001 0.001 0.001
- link back_long_arm_arm: geometry collision box size=0.35 0.05 0.30; visual mesh filename=file:///home/oli/ros2_ws/install/rocap_ros/share/rocap_ros/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 scale=0.001 0.001 0.001
- link back_short_arm_1_arm: geometry collision box size=0.16 0.05 0.20; visual mesh filename=file:///home/oli/ros2_ws/install/rocap_ros/share/rocap_ros/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 scale=0.001 0.001 0.001
- link back_short_arm_2_arm: geometry collision box size=0.16 0.05 0.20; visual mesh filename=file:///home/oli/ros2_ws/install/rocap_ros/share/rocap_ros/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 scale=0.001 0.001 0.001
- link base_link: geometry 
- link front_long_arm_arm: geometry collision box size=0.35 0.05 0.30; visual mesh filename=file:///home/oli/ros2_ws/install/rocap_ros/share/rocap_ros/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 scale=0.001 0.001 0.001
- link front_short_arm_1_arm: geometry collision box size=0.16 0.05 0.20; visual mesh filename=file:///home/oli/ros2_ws/install/rocap_ros/share/rocap_ros/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 scale=0.001 0.001 0.001
- link front_short_arm_2_arm: geometry collision box size=0.16 0.05 0.20; visual mesh filename=file:///home/oli/ros2_ws/install/rocap_ros/share/rocap_ros/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 scale=0.001 0.001 0.001
- link left_long_arm_arm: geometry collision box size=0.35 0.05 0.30; visual mesh filename=file:///home/oli/ros2_ws/install/rocap_ros/share/rocap_ros/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 scale=0.001 0.001 0.001
- link left_short_arm_1_arm: geometry collision box size=0.16 0.05 0.20; visual mesh filename=file:///home/oli/ros2_ws/install/rocap_ros/share/rocap_ros/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 scale=0.001 0.001 0.001
- link left_short_arm_2_arm: geometry collision box size=0.16 0.05 0.20; visual mesh filename=file:///home/oli/ros2_ws/install/rocap_ros/share/rocap_ros/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 scale=0.001 0.001 0.001
- link right_long_arm_arm: geometry collision box size=0.35 0.05 0.30; visual mesh filename=file:///home/oli/ros2_ws/install/rocap_ros/share/rocap_ros/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 scale=0.001 0.001 0.001
- link right_short_arm_1_arm: geometry collision box size=0.16 0.05 0.20; visual mesh filename=file:///home/oli/ros2_ws/install/rocap_ros/share/rocap_ros/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 scale=0.001 0.001 0.001
- link right_short_arm_2_arm: geometry collision box size=0.16 0.05 0.20; visual mesh filename=file:///home/oli/ros2_ws/install/rocap_ros/share/rocap_ros/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 scale=0.001 0.001 0.001
Joints:
- removed joint base_link_to_back_rotation_link
- removed joint base_link_to_front_rotation_link
- removed joint base_link_to_left_rotation_link
- removed joint base_link_to_lidar_base_link
- removed joint base_link_to_right_rotation_link
- added joint rocap_body_j: type fixed, parent base_link, child rocap_body, origin xyz=0 0 0 rpy=0 0 0
- added joint rocap_body_to_back_rotation_link: type fixed, parent rocap_body, child back_rotation_link, origin xyz=0 0 0 rpy=0 0 3.141592653589793
- added joint rocap_body_to_front_rotation_link: type fixed, parent rocap_body, child front_rotation_link, origin xyz=0 0 0 rpy=0 0 0.0
- added joint rocap_body_to_left_rotation_link: type fixed, parent rocap_body, child left_rotation_link, origin xyz=0 0 0 rpy=0 0 1.5707963267948966
- added joint rocap_body_to_lidar_base_link: type fixed, parent rocap_body, child lidar_base_link, origin xyz=-.15 -0.150 0 rpy=3.141592653589793 0 0
- added joint rocap_body_to_right_rotation_link: type fixed, parent rocap_body, child right_rotation_link, origin xyz=0 0 0 rpy=0 0 4.71238898038469

File: rocap_ros/urdf/rocap_body/rocap_body.urdf.xacro (robot description, xacro)
@@ -151,8 +151,8 @@
     <xacro:all_side_arm name="right" fix_to_link="base_link" angleZ="${pi/2*3}" fixed_arm="${fixed_arm}" />
     <!-- add sensor -->
-    <xacro:include filename="$(find cta_gazebo_part)/part/movement/moving_base_6_axis/moving_base_6_axis.urdf.xacro" />
-    <xacro:include filename="$(find cta_gazebo_part)/part/lidar/velodyme_puck/velodyme_puck.urdf.xacro" />
-    <xacro:include filename="$(find cta_gazebo_part)/part/IMU/IMU.urdf.xacro" />
-    <xacro:include filename="$(find cta_gazebo_part)/part/camera/cameraDepth/cameraDepth.urdf.xacro" />
+    <xacro:include filename="$(find rocap_ros)/urdf/part/movement/moving_base_6_axis/moving_base_6_axis.urdf.xacro" />
+    <xacro:include filename="$(find rocap_ros)/urdf/part/lidar/velodyme_puck/velodyme_puck.urdf.xacro" />
+    <xacro:include filename="$(find rocap_ros)/urdf/part/IMU/IMU.urdf.xacro" />
+    <xacro:include filename="$(find rocap_ros)/urdf/part/camera/cameraDepth/cameraDepth.urdf.xacro" />
     <xacro:velodyme_puck namespace="/ray" fixTo="base_link" fixToBaseXYZ="-.15 -0.150 0" fixToBaseRPY="${pi} 0 0"/>
     <xacro:IMU name="IMU" fix_to="base_link" xyz="0 0 0" rpy="0 0 0"/>

File: rocap_ros/urdf/rocap_flying_demo/rocap_flying_demo.urdf (robot description, URDF)
Before this commit: robot flying_rocap_body, 73 links, 72 joints
Links:
- added link rocap_body, mass 0.001; collision box size=0.4 0.4 0.45; visual mesh filename=file:///home/oli/ros2_ws/install/rocap_ros/share/rocap_ros/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 scale=0.001 0.001 0.001
- link back_long_arm_arm: geometry collision box size=0.35 0.05 0.30; visual mesh filename=file:///home/oli/ros2_ws/install/rocap_ros/share/rocap_ros/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 scale=0.001 0.001 0.001
- link back_short_arm_1_arm: geometry collision box size=0.16 0.05 0.20; visual mesh filename=file:///home/oli/ros2_ws/install/rocap_ros/share/rocap_ros/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 scale=0.001 0.001 0.001
- link back_short_arm_2_arm: geometry collision box size=0.16 0.05 0.20; visual mesh filename=file:///home/oli/ros2_ws/install/rocap_ros/share/rocap_ros/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 scale=0.001 0.001 0.001
- link base_A_ancor_module_center: geometry visual mesh filename=file:///home/oli/ros2_ws/install/rocap_ros/share/rocap_ros/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 scale=0.001 0.001 0.001
- link base_A_ancor_module_left: geometry visual mesh filename=file:///home/oli/ros2_ws/install/rocap_ros/share/rocap_ros/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 scale=0.001 0.001 0.001
- link base_A_ancor_module_right: geometry visual mesh filename=file:///home/oli/ros2_ws/install/rocap_ros/share/rocap_ros/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 scale=0.001 0.001 0.001
- link base_B_ancor_module_center: geometry visual mesh filename=file:///home/oli/ros2_ws/install/rocap_ros/share/rocap_ros/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 scale=0.001 0.001 0.001
- link base_B_ancor_module_left: geometry visual mesh filename=file:///home/oli/ros2_ws/install/rocap_ros/share/rocap_ros/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 scale=0.001 0.001 0.001
- link base_B_ancor_module_right: geometry visual mesh filename=file:///home/oli/ros2_ws/install/rocap_ros/share/rocap_ros/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 scale=0.001 0.001 0.001
- link base_C_ancor_module_center: geometry visual mesh filename=file:///home/oli/ros2_ws/install/rocap_ros/share/rocap_ros/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 scale=0.001 0.001 0.001
- link base_C_ancor_module_left: geometry visual mesh filename=file:///home/oli/ros2_ws/install/rocap_ros/share/rocap_ros/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 scale=0.001 0.001 0.001
- link base_C_ancor_module_right: geometry visual mesh filename=file:///home/oli/ros2_ws/install/rocap_ros/share/rocap_ros/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 scale=0.001 0.001 0.001
- link base_D_ancor_module_center: geometry visual mesh filename=file:///home/oli/ros2_ws/install/rocap_ros/share/rocap_ros/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 scale=0.001 0.001 0.001
- link base_D_ancor_module_left: geometry visual mesh filename=file:///home/oli/ros2_ws/install/rocap_ros/share/rocap_ros/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 scale=0.001 0.001 0.001
- link base_D_ancor_module_right: geometry visual mesh filename=file:///home/oli/ros2_ws/install/rocap_ros/share/rocap_ros/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 scale=0.001 0.001 0.001
- link base_link: geometry 
- link front_long_arm_arm: geometry collision box size=0.35 0.05 0.30; visual mesh filename=file:///home/oli/ros2_ws/install/rocap_ros/share/rocap_ros/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 scale=0.001 0.001 0.001
- link front_short_arm_1_arm: geometry collision box size=0.16 0.05 0.20; visual mesh filename=file:///home/oli/ros2_ws/install/rocap_ros/share/rocap_ros/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 scale=0.001 0.001 0.001
- link front_short_arm_2_arm: geometry collision box size=0.16 0.05 0.20; visual mesh filename=file:///home/oli/ros2_ws/install/rocap_ros/share/rocap_ros/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 scale=0.001 0.001 0.001
- link left_long_arm_arm: geometry collision box size=0.35 0.05 0.30; visual mesh filename=file:///home/oli/ros2_ws/install/rocap_ros/share/rocap_ros/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 scale=0.001 0.001 0.001
- link left_short_arm_1_arm: geometry collision box size=0.16 0.05 0.20; visual mesh filename=file:///home/oli/ros2_ws/install/rocap_ros/share/rocap_ros/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 scale=0.001 0.001 0.001
- link left_short_arm_2_arm: geometry collision box size=0.16 0.05 0.20; visual mesh filename=file:///home/oli/ros2_ws/install/rocap_ros/share/rocap_ros/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 scale=0.001 0.001 0.001
- link right_long_arm_arm: geometry collision box size=0.35 0.05 0.30; visual mesh filename=file:///home/oli/ros2_ws/install/rocap_ros/share/rocap_ros/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 scale=0.001 0.001 0.001
- link right_short_arm_1_arm: geometry collision box size=0.16 0.05 0.20; visual mesh filename=file:///home/oli/ros2_ws/install/rocap_ros/share/rocap_ros/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 scale=0.001 0.001 0.001
- link right_short_arm_2_arm: geometry collision box size=0.16 0.05 0.20; visual mesh filename=file:///home/oli/ros2_ws/install/rocap_ros/share/rocap_ros/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 scale=0.001 0.001 0.001
Joints:
- removed joint base_link_to_back_rotation_link
- removed joint base_link_to_front_rotation_link
- removed joint base_link_to_left_rotation_link
- removed joint base_link_to_lidar_base_link
- removed joint base_link_to_right_rotation_link
- added joint rocap_body_j: type fixed, parent base_link, child rocap_body, origin xyz=0 0 0 rpy=0 0 0
- added joint rocap_body_to_back_rotation_link: type fixed, parent rocap_body, child back_rotation_link, origin xyz=0 0 0 rpy=0 0 3.141592653589793
- added joint rocap_body_to_front_rotation_link: type fixed, parent rocap_body, child front_rotation_link, origin xyz=0 0 0 rpy=0 0 0.0
- added joint rocap_body_to_left_rotation_link: type fixed, parent rocap_body, child left_rotation_link, origin xyz=0 0 0 rpy=0 0 1.5707963267948966
- added joint rocap_body_to_lidar_base_link: type fixed, parent rocap_body, child lidar_base_link, origin xyz=-.15 -0.150 0 rpy=3.141592653589793 0 0
- added joint rocap_body_to_right_rotation_link: type fixed, parent rocap_body, child right_rotation_link, origin xyz=0 0 0 rpy=0 0 4.71238898038469
- joint lin_x: limit lower=-10000 upper=10000 effort=1000 velocity=0.5 -> lower=-10000 upper=10000 effort=1000 velocity=30
- joint lin_y: limit lower=-10000 upper=10000 effort=1000 velocity=0.5 -> lower=-10000 upper=10000 effort=1000 velocity=30
- joint lin_z: limit lower=-10000 upper=10000 effort=1000 velocity=0.5 -> lower=-10000 upper=10000 effort=1000 velocity=30
- joint rot_x: limit lower=10000 upper=10000 effort=10000.0 velocity=0.5 -> lower=10000 upper=10000 effort=1000000000000000.0 velocity=30
- joint rot_y: limit lower=10000 upper=10000 effort=10000.0 velocity=0.5 -> lower=10000 upper=10000 effort=1000000000000000.0 velocity=30
- joint rot_z: limit lower=10000 upper=10000 effort=10000.0 velocity=0.5 -> lower=10000 upper=10000 effort=1000000000000000.0 velocity=30

File: rocap_ros/urdf/rocap_flying_demo/rocap_flying_demo.urdf.xacro (robot description, xacro)
@@ -6,5 +6,5 @@
   <xacro:property name="package" value="rocap_ros" />
   <!-- define all file include -->
-  <xacro:include filename="$(find cta_gazebo_part)/part/movement/moving_base_6_axis/moving_base_6_axis.urdf.xacro" />
+  <xacro:include filename="$(find rocap_ros)/urdf/part/movement/moving_base_6_axis/moving_base_6_axis.urdf.xacro" />
   <xacro:include filename="$(find rocap_ros)/urdf/rocap_body/rocap_body.urdf.xacro"/>
   <xacro:include filename="$(find rocap_ros)/urdf/rocap_base/rocap_base.urdf.xacro"/>
@@ -22,5 +22,5 @@
                             initial_position_lin_x="-2"
                             initial_position_lin_y="4.5"
-                            initial_position_lin_z="2"
+                            initial_position_lin_z="5"
                             initial_position_rot_z="${3*pi/4}"
                             lin_x_vel_kp="1000"
